File: sprinklers.kicad_pcb (KiCad board)
At the start: 2 copper layers, 147.3 x 78.7 mm, 67 parts, among them J1 Conn_01x02, J2 Conn_01x02, J3 Conn_01x02, J4 Conn_01x02, J5 Conn_01x02, J6 Conn_01x02, J8 Conn_01x04_Pin, J9 Conn_01x03_Pin, K1 SANYOU_SRD_Form_C, K2 SANYOU_SRD_Form_C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

Commit message: fix EN net
Connections:
- PROG/EXT1 pad 6: Net-(PROG/EXT1-Pin_6) -> Net-(J11-Pin_1)
- U2 pad 3: Net-(PROG/EXT1-Pin_6) -> Net-(J11-Pin_1)
Routing:
- net Net-(J11-Pin_1): track 85.1 -> 72.6 mm, vias 0 -> 1
Changed lines of the file:
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@@
       (net 6 "3V3") (pinfunction "VDD") (pintype "power_in"))
     (pad "3" smd rect (at -8.75 -5.71 270) (size 1.5 0.9) (layers "F.Cu" "F.Paste" "F.Mask")
-      (net 74 "Net-(PROG/EXT1-Pin_6)") (pinfunction "EN") (pintype "input"))
+      (net 17 "Net-(J11-Pin_1)") (pinfunction "EN") (pintype "input"))
     (pad "4" smd rect (at -8.75 -4.44 270) (size 1.5 0.9) (layers "F.Cu" "F.Paste" "F.Mask")
       (net 18 "unconnected-(U2-SENSOR_VP-Pad4)") (pinfunction "SENSOR_VP") (pintype "input"))
@@
       (net 71 "Net-(PROG/EXT1-Pin_5)") (pinfunction "Pin_5") (pintype "passive"))
     (pad "6" thru_hole oval (at 0 12.7 270) (size 1.7 1.7) (drill 1) (layers "*.Cu" "*.Mask")
-      (net 74 "Net-(PROG/EXT1-Pin_6)") (pinfunction "Pin_6") (pintype "passive"))
+      (net 17 "Net-(J11-Pin_1)") (pinfunction "Pin_6") (pintype "passive"))
     (model "${KICAD6_3DMODEL_DIR}/Connector_PinHeader_2.54mm.3dshapes/PinHeader_1x06_P2.54mm_Vertical.wrl"
       (offset (xyz 0 0 0))
@@
   (segment (start 121.131 45.6898) (end 121.131 46.1532) (width 0.25) (layer "F.Cu") (net 16))
   (segment (start 137.16 65.8475) (end 137.362 66.05) (width 0.25) (layer "F.Cu") (net 17))
+  (segment (start 144.716506 32.047494) (end 144.18735 32.047494) (width 0.25) (layer "F.Cu") (net 17))
   (segment (start 147.177 66.05) (end 147.878 66.7511) (width 0.25) (layer "F.Cu") (net 17))
-  (segment (start 146.02 28.9171) (end 138.1371 28.9171) (width 0.25) (layer "F.Cu") (net 17))
-  (segment (start 146.02 29.994) (end 146.02 28.9171) (width 0.25) (layer "F.Cu") (net 17))
+  (segment (start 146.02 29.994) (end 146.02 30.744) (width 0.25) (layer "F.Cu") (net 17))
   (segment (start 146 66.05) (end 147.177 66.05) (width 0.25) (layer "F.Cu") (net 17))
-  (segment (start 138.1371 28.9171) (end 133.35 24.13) (width 0.25) (layer "F.Cu") (net 17))
+  (segment (start 146.02 30.744) (end 144.716506 32.047494) (width 0.25) (layer "F.Cu") (net 17))
   (segment (start 137.362 66.05) (end 139.7 66.05) (width 0.25) (layer "F.Cu") (net 17))
   (segment (start 139.7 66.05) (end 146 66.05) (width 0.25) (layer "F.Cu") (net 17))
   (segment (start 147.878 66.7511) (end 149.86 66.7511) (width 0.25) (layer "F.Cu") (net 17))
+  (via (at 144.18735 32.047494) (size 0.8) (drill 0.4) (layers "F.Cu" "B.Cu") (net 17))
+  (segment (start 144.18735 32.12105) (end 147.409067 35.342767) (width 0.25) (layer "B.Cu") (net 17))
   (segment (start 148.10117 36.034489) (end 148.10117 63.300958) (width 0.25) (layer "B.Cu") (net 17))
   (segment (start 140.992 22.4342) (end 142.165 23.6071) (width 0.25) (layer "B.Cu") (net 17))
-  (segment (start 142.165 30.0987) (end 147.409067 35.342767) (width 0.25) (layer "B.Cu") (net 17))
+  (segment (start 144.113794 32.047494) (end 144.18735 32.047494) (width 0.25) (layer "B.Cu") (net 17))
+  (segment (start 142.165 30.0987) (end 144.113794 32.047494) (width 0.25) (layer "B.Cu") (net 17))
   (segment (start 147.409067 35.342767) (end 147.409448 35.342767) (width 0.25) (layer "B.Cu") (net 17))
   (segment (start 147.409448 35.342767) (end 148.10117 36.034489) (width 0.25) (layer "B.Cu") (net 17))
@@
   (segment (start 142.165 23.6071) (end 142.165 30.0987) (width 0.25) (layer "B.Cu") (net 17))
   (segment (start 135.046 22.4342) (end 140.992 22.4342) (width 0.25) (layer "B.Cu") (net 17))
+  (segment (start 144.18735 32.047494) (end 144.18735 32.12105) (width 0.25) (layer "B.Cu") (net 17))
   (segment (start 133.35 24.13) (end 135.046 22.4342) (width 0.25) (layer "B.Cu") (net 17))
   (segment (start 148.10117 63.300958) (end 149.86 65.059788) (width 0.25) (layer "B.Cu") (net 17))
