File: controller/sprinklers.kicad_sch (KiCad schematic)
At the start: 66 parts, among them J1 Conn_01x02, J2 Conn_01x02, J3 Conn_01x02, J4 Conn_01x02, J5 Conn_01x02, J6 Conn_01x02, J8 Conn_01x04_Pin, J9 Conn_01x03_Pin, K1 SANYOU_SRD_Form_C, K2 SANYOU_SRD_Form_C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

Commit message: Rel V1.2
Parts:
- removed J9: Conn_01x03_Pin, Connector_PinHeader_2.54mm:PinHeader_1x03_P2.54mm_Vertical, symbol Connector:Conn_01x03_Pin
- removed PROG/EXT1: Conn_01x06_Pin, Connector_PinHeader_2.54mm:PinHeader_1x06_P2.54mm_Vertical, symbol Connector:Conn_01x06_Pin
- removed R10, R6, R7, R8, R9: 1K, Resistor_SMD:R_1206_3216Metric, symbol Device:R
- removed RST1: Conn_01x02_Pin, Connector_PinHeader_2.54mm:PinHeader_1x02_P2.54mm_Vertical, symbol Connector:Conn_01x02_Pin
- added POWER1, PROG1: Conn_01x04_Pin, Connector_JST:JST_PH_B4B-PH-K_1x04_P2.00mm_Vertical, symbol Connector:Conn_01x04_Pin
- added R5 (x5): 10K, Resistor_SMD:R_1206_3216Metric, symbol Device:R
- C1: LCSC C52923 -> C440198
- D1: footprint LED_SMD:LED_0402_1005Metric -> LED_SMD:LED_0805_2012Metric; LCSC C130721 -> C2286
- D2: footprint LED_SMD:LED_0402_1005Metric -> LED_SMD:LED_0805_2012Metric; LCSC C130719 -> C2296
- D3: footprint LED_SMD:LED_0402_1005Metric -> LED_SMD:LED_0603_1608Metric; LCSC C130724 -> C2297
- EXT1: footprint Connector_PinHeader_2.54mm:PinHeader_1x04_P2.54mm_Vertical -> Connector_JST:JST_PH_B4B-PH-K_1x04_P2.00mm_Vertical
- LED1: renamed from J8; footprint Connector_PinHeader_2.54mm:PinHeader_1x04_P2.54mm_Vertical -> Connector_JST:JST_PH_B4B-PH-K_1x04_P2.00mm_Vertical
- R5: value 1K -> 10K; LCSC C4410 -> C17902
- RST_SW1: LCSC (none) -> C318884
- U2: value ESP32-WROOM-32D -> ESP32-WROOM-32U; footprint RF_Module:ESP32-WROOM-32D -> RF_Module:ESP32-WROOM-32U; LCSC C529577 -> C328062
Connections:
- net 3V3: now also POWER1.3 (Pin_3)
- net 5V: now also POWER1.2 (Pin_2)
- net GND1: now also POWER1.4 (Pin_4), R5.2, R5.2, R5.2, R5.2, R5.2
- net at K1.2: now also D14.2 (A); no longer D14.1 (K)
- net at Q5.1 (G), U2.13 (IO14): now also R5.1
- net at Q4.1 (G), U2.12 (IO27): now also R5.1
- net at Q3.1 (G), U2.11 (IO26): now also R5.1
- net at D11.1 (K): now also Q1.2 (D); no longer K2.2
- net at D11.2 (A): now also K2.2; no longer Q1.2 (D)
- net at R6.2, RST_SW1.1 (A), U2.3 (EN): now also POWER1.1 (Pin_1), PROG1.4 (Pin_4)
- net at D13.1 (K): now also Q5.2 (D); no longer K6.2
- net at D13.2 (A): now also K6.2; no longer Q5.2 (D)
- net at D12.1 (K): now also Q4.2 (D); no longer K5.2
- net at D12.2 (A): now also K5.2; no longer Q4.2 (D)
- net at Q2.1 (G), U2.10 (IO25): now also R5.1
- net at Q2.2 (D): now also D10.1 (K); no longer D10.2 (A)
- net at U2.25 (IO0): now also PROG1.1 (Pin_1)
- net at U2.34 (RXD0/IO3): now also PROG1.2 (Pin_2)
- net at U2.35 (TXD0/IO1): now also PROG1.3 (Pin_3)
- net at Q6.1 (G), U2.14 (IO12): now also R5.1
- net at Q6.2 (D): now also D14.1 (K); no longer D14.2 (A)
- net at K3.2: now also D10.2 (A); no longer D10.1 (K)
- net at D9.1 (K): now also Q3.2 (D); no longer K4.2
- net at D9.2 (A): now also K4.2; no longer Q3.2 (D)
Other:
- moved on the sheet: D10, D11, D12, D13, D14, D9, R6

Commit message: fix footprint
Parts:
- C1: footprint Capacitor_SMD:C_0402_1005Metric -> Capacitor_SMD:C_0805_2012Metric
- R1: footprint Resistor_SMD:R_0201_0603Metric -> Resistor_SMD:R_0603_1608Metric
Changed lines of the file:
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@@
       (effects (font (size 1.27 1.27)) hide)
     )
-    (property "Footprint" "Resistor_SMD:R_0201_0603Metric" (at 167.005 87.122 90)
+    (property "Footprint" "Resistor_SMD:R_0603_1608Metric" (at 167.005 87.122 90)
       (effects (font (size 1.27 1.27)) hide)
     )
@@
       (effects (font (size 1.27 1.27)) hide)
     )
-    (property "Footprint" "Resistor_SMD:R_0201_0603Metric" (at 158.75 64.262 90)
+    (property "Footprint" "Resistor_SMD:R_0603_1608Metric" (at 158.75 64.262 90)
       (effects (font (size 1.27 1.27)) hide)
     )
@@
       (effects (font (size 1.27 1.27)) hide)
     )
-    (property "Footprint" "Resistor_SMD:R_0201_0603Metric" (at 167.005 75.692 90)
+    (property "Footprint" "Resistor_SMD:R_0603_1608Metric" (at 167.005 75.692 90)
       (effects (font (size 1.27 1.27)) hide)
     )
@@
       (effects (font (size 1.27 1.27)) hide)
     )
-    (property "Footprint" "Resistor_SMD:R_0201_0603Metric" (at 158.75 67.437 90)
+    (property "Footprint" "Resistor_SMD:R_0603_1608Metric" (at 158.75 67.437 90)
       (effects (font (size 1.27 1.27)) hide)
     )
@@
       (effects (font (size 1.27 1.27)) (justify left) hide)
     )
-    (property "Footprint" "Capacitor_SMD:C_0402_1005Metric" (at 30.48 53.0352 0)
+    (property "Footprint" "Capacitor_SMD:C_0805_2012Metric" (at 30.48 53.0352 0)
       (effects (font (size 1.27 1.27)) hide)
     )
@@
       (effects (font (size 1.27 1.27)) hide)
     )
-    (property "Footprint" "Resistor_SMD:R_0201_0603Metric" (at 167.005 81.407 90)
+    (property "Footprint" "Resistor_SMD:R_0603_1608Metric" (at 167.005 81.407 90)
       (effects (font (size 1.27 1.27)) hide)
     )
@@
       (effects (font (size 1.27 1.27)) (justify left) hide)
     )
-    (property "Footprint" "Capacitor_SMD:C_0402_1005Metric" (at 27.94 85.4202 0)
+    (property "Footprint" "Capacitor_SMD:C_0805_2012Metric" (at 27.94 85.4202 0)
       (effects (font (size 1.27 1.27)) hide)
     )
@@
       (effects (font (size 1.27 1.27)) hide)
     )
-    (property "Footprint" "Resistor_SMD:R_0201_0603Metric" (at 158.75 61.087 90)
-      (effects (font (size 1.27 1.27)) hide)
-    )
+    (property "Footprint" "Resistor_SMD:R_0603_1608Metric" (at 158.75 61.087 90)
+      (effects (font (size 1.27 1.27)) hide)
+    )
