File: sensor/moisture.kicad_sch (KiCad schematic)
At the start: 35 parts, among them U1 LM2596S-5, U2 ESP32-WROOM-32U, U3 AP1117-33

Commit message: fix footprint
Parts:
- C1: footprint Capacitor_SMD:C_0402_1005Metric -> Capacitor_SMD:C_0805_2012Metric
- R1: footprint Resistor_SMD:R_0201_0603Metric -> Resistor_SMD:R_0603_1608Metric
Changed lines of the file:
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@@
       (effects (font (size 1.27 1.27)) hide)
     )
-    (property "Footprint" "Resistor_SMD:R_0201_0603Metric" (at 167.005 87.122 90)
+    (property "Footprint" "Resistor_SMD:R_0603_1608Metric" (at 167.005 87.122 90)
       (effects (font (size 1.27 1.27)) hide)
     )
@@
       (effects (font (size 1.27 1.27)) hide)
     )
-    (property "Footprint" "Resistor_SMD:R_0201_0603Metric" (at 158.75 64.262 90)
+    (property "Footprint" "Resistor_SMD:R_0603_1608Metric" (at 158.75 64.262 90)
       (effects (font (size 1.27 1.27)) hide)
     )
@@
       (effects (font (size 1.27 1.27)) hide)
     )
-    (property "Footprint" "Resistor_SMD:R_0201_0603Metric" (at 167.005 75.692 90)
+    (property "Footprint" "Resistor_SMD:R_0603_1608Metric" (at 167.005 75.692 90)
       (effects (font (size 1.27 1.27)) hide)
     )
@@
       (effects (font (size 1.27 1.27)) hide)
     )
-    (property "Footprint" "Resistor_SMD:R_0201_0603Metric" (at 158.75 67.437 90)
+    (property "Footprint" "Resistor_SMD:R_0603_1608Metric" (at 158.75 67.437 90)
       (effects (font (size 1.27 1.27)) hide)
     )
@@
       (effects (font (size 1.27 1.27)) (justify left) hide)
     )
-    (property "Footprint" "Capacitor_SMD:C_0402_1005Metric" (at 30.48 53.0352 0)
+    (property "Footprint" "Capacitor_SMD:C_0805_2012Metric" (at 30.48 53.0352 0)
       (effects (font (size 1.27 1.27)) hide)
     )
@@
       (effects (font (size 1.27 1.27)) hide)
     )
-    (property "Footprint" "Resistor_SMD:R_0201_0603Metric" (at 167.005 81.407 90)
+    (property "Footprint" "Resistor_SMD:R_0603_1608Metric" (at 167.005 81.407 90)
       (effects (font (size 1.27 1.27)) hide)
     )
@@
       (effects (font (size 1.27 1.27)) (justify left) hide)
     )
-    (property "Footprint" "Capacitor_SMD:C_0402_1005Metric" (at 27.94 85.4202 0)
+    (property "Footprint" "Capacitor_SMD:C_0805_2012Metric" (at 27.94 85.4202 0)
       (effects (font (size 1.27 1.27)) hide)
     )
@@
       (effects (font (size 1.27 1.27)) hide)
     )
-    (property "Footprint" "Resistor_SMD:R_0201_0603Metric" (at 158.75 61.087 90)
-      (effects (font (size 1.27 1.27)) hide)
-    )
+    (property "Footprint" "Resistor_SMD:R_0603_1608Metric" (at 158.75 61.087 90)
+      (effects (font (size 1.27 1.27)) hide)
+    )
